File: door_unlocker.sch (EAGLE design)
At the start: 16 parts, among them IC1 LM2937, T1 2N3904

Commit message: de-clusterfucked the schematic.
Parts:
- removed POWER_SEL: (no value), adafruit:PINHD-1X3
- added T2: 2N3904, transistor:2N3904
Connections:
- net N$2 renamed 5V
- net N$9 renamed SERVO_SIGNAL
- net RX renamed FTDI_RX_8266_TX
- net TX renamed FTDI_TX_8266_RX
- removed net 8266_3P3V: EN_R.1, ESP8266.7, POWER_SEL.2
- removed net N$3: C2.+, IC1.VO, POWER_SEL.3, SW1.P$1
- removed net N$5: SERVO.1, T1.C
- new net FTDI_3P3V: FTDI.4
- new net SERVO_GND: SERVO.1, T1.C, T2.C
- net 3P3V: now also C2.+, EN_R.1, ESP8266.7, IC1.VO; no longer FTDI.4, POWER_SEL.1
- net GND: now also SW1.P$1, T2.E
- net N$8: now also T2.B
Other:
- note added: "Pull GPIO0 down to program. Pull up GPIO0 and GPIO2 to run."
- moved on the sheet: C1, C2, CN1, EN_R, FTDI, GPIO0, GPIO2, IC1, R1, R2, R3, SERVO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

Commit message: added servo status LED.
Parts:
- added LED1: (no value), led:LED5MM
- added R4: 100, resistor:R-US_0207/10
Connections:
- new net N$2: LED1.A, R4.1
- net GND: now also LED1.C
- net N$7: now also R4.2
Changed lines of the file:
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@@
 <part name="GND11" library="supply1" deviceset="GND" device=""/>
 <part name="GND12" library="supply1" deviceset="GND" device=""/>
+<part name="R4" library="resistor" deviceset="R-US_" device="0207/10" value="100"/>
+<part name="LED1" library="led" deviceset="LED" device="5MM"/>
+<part name="GND6" library="supply1" deviceset="GND" device=""/>
 </parts>
 <sheets>
@@
 <instance part="GND11" gate="1" x="124.46" y="76.2"/>
 <instance part="GND12" gate="1" x="124.46" y="50.8"/>
+<instance part="R4" gate="G$1" x="147.32" y="35.56" rot="R90"/>
+<instance part="LED1" gate="G$1" x="147.32" y="27.94"/>
+<instance part="GND6" gate="1" x="147.32" y="17.78"/>
 </instances>
 <busses>
@@
 <pinref part="SW1" gate="G$1" pin="P$1"/>
 <wire x1="53.34" y1="20.32" x2="53.34" y2="22.86" width="0.1524" layer="91"/>
+</segment>
+<segment>
+<pinref part="GND6" gate="1" pin="GND"/>
+<pinref part="LED1" gate="G$1" pin="C"/>
+<wire x1="147.32" y1="20.32" x2="147.32" y2="22.86" width="0.1524" layer="91"/>
 </segment>
 </net>
@@
 <pinref part="GPIO0" gate="A" pin="3"/>
 <pinref part="R1" gate="G$1" pin="1"/>
-<wire x1="114.3" y1="43.18" x2="162.56" y2="43.18" width="0.1524" layer="91"/>
+<wire x1="114.3" y1="43.18" x2="147.32" y2="43.18" width="0.1524" layer="91"/>
+<pinref part="R4" gate="G$1" pin="2"/>
+<wire x1="147.32" y1="43.18" x2="162.56" y2="43.18" width="0.1524" layer="91"/>
+<wire x1="147.32" y1="40.64" x2="147.32" y2="43.18" width="0.1524" layer="91"/>
+<junction x="147.32" y="43.18"/>
 </segment>
 </net>
@@
 </segment>
 </net>
+<net name="N$2" class="0">
+<segment>
+<pinref part="R4" gate="G$1" pin="1"/>
+<pinref part="LED1" gate="G$1" pin="A"/>
+</segment>
+</net>
